Commit message: patched iiwa_hw (new controller), iiwa_moveit(for sensors and planning) iiwa_description(gripper and flange)

File: iiwa_description/urdf/iiwa7.xacro (robot description, xacro)
@@ -268,5 +268,6 @@
       <inertial>
         <origin xyz="0 0 0.02" rpy="0 0 0"/>
-        <mass value="3.129"/>
+<!--       <mass value="3.129"/> Original from iiwwa_stack-->
+        <mass value="0.458"/>
         <inertia ixx="0.01464"  ixy="0.0005912"  ixz="0" iyy="0.01465" iyz="0" izz="0.002872" />
       </inertial>
@@ -274,5 +275,5 @@
         <origin xyz="0 0 -0.0005" rpy="0 0 0"/>
         <geometry>
-          <mesh filename="package://iiwa_description/meshes/iiwa7/visual/link_7.stl"/>
+          <mesh filename="package://iiwa_description/meshes/iiwa7/visual/link_7_pneumatic.stl" scale="0.001 0.001 0.001"/>
         </geometry>
         <material name="Grey"/>
@@ -281,5 +282,5 @@
         <origin xyz="0 0 -0.0005" rpy="0 0 0"/>
         <geometry>
-          <mesh filename="package://iiwa_description/meshes/iiwa7/collision/link_7.stl"/>
+          <mesh filename="package://iiwa_description/meshes/iiwa7/collision/link_7_pneumatic.stl" scale="0.001 0.001 0.001"/>
         </geometry>
         <material name="Grey"/>
@@ -289,8 +290,45 @@
       <parent link="${robot_name}_link_7"/>
       <child link="${robot_name}_link_ee"/>
-      <origin xyz="0 0 0.045" rpy="0 0 0"/>
+      <origin xyz="0 0 0.071" rpy="0 0 0"/>
+      <!-- Distanza di hand effector visualizzato in rviz come una sfera azzurra, attaccato al liink7 -->
     </joint>
     <link name="${robot_name}_link_ee">
     </link>
+    <!--  Here we define a dummy joint between the tip of the iiwa7 and the base of the tool.
+      There is no offset between the two, that means the tool is attached to the robot flange. -->
+    <joint name="tool_joint" type="fixed">
+      <parent link="${robot_name}_link_ee" />
+      <child link = "tool_link" />
+      <origin xyz="0 0 0" rpy="0 0 0" />
+    </joint>
+    <!-- Here we define the geometry of the tool. We designed the tool ourselves, so we have a mesh file that represents it.
+      Else, one can define it using a geometric representation that approximate it, like a cylinder (see commented lines) -->
+    <link name="tool_link">
+      <visual>
+        <origin xyz="0 0 -0.001" rpy="0 0 0"/>
+        <geometry>
+          <mesh filename="package://iiwa_description/meshes/iiwa7/visual/3fingersleppaG.stl" scale="0.001 0.001 0.001"/>
+          <!-- 	<cylinder length="0.1275" radius="0.020"/> -->
+        </geometry>
+        <material name="Grey"/>
+      </visual>
+      <collision>
+        <origin xyz="0 0 -0.001" rpy="0 0 0"/>
+        <geometry>
+          <mesh filename="package://iiwa_description/meshes/iiwa7/visual/3fingersleppaG.stl" scale="0.001 0.001 0.001"/>
+        <!-- 	<cylinder length="0.1275" radius="0.020"/> -->
+        </geometry>
+        <material name="Grey"/>
+      </collision>
+    </link>
+      <!--  Here we define another dummy joint.
+    It is placed at the end of the tool (12.75 cm), so we can then attach a frame at its TCP for control -->
+    <joint name="tool_tip_joint" type="fixed">
+      <parent link="tool_link" />
+      <child link = "tool_link_ee" />
+      <origin xyz="0 0 0.125" rpy="0 0 0" />
+    </joint>
+    <!--  The TCP frame is here defined -->
+    <link name="tool_link_ee"/>
     <!--Extensions -->
     <xacro:iiwa_gazebo robot_name="${robot_name}" />
